File: brick_sorter/Board/psu.sch (EAGLE design)
At the start: 14 parts, among them IC1 LM2574N-3.3, IC2-12V 786TV, IC2-6V 786TV

Commit message: Board v2.0
Connections:
- net N$2 renamed LM_OUT
Changed lines of the file:
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@@
 <part name="C1" library="rcl" deviceset="CPOL-US" device="E5-8.5"/>
 <part name="C2" library="rcl" deviceset="CPOL-US" device="E5-5"/>
-<part name="L1" library="inductor-neosid" deviceset="BS" device="11"/>
 <part name="D1" library="diode" deviceset="BYV10" device=""/>
 <part name="SL1" library="con-amp-quick" deviceset="M10" device=""/>
@@
 <part name="D3" library="diode" deviceset="1N4004" device=""/>
 <part name="C6" library="rcl" deviceset="C-EU" device="050-030X075"/>
+<part name="L1" library="inductor-neosid" deviceset="BS" device="11"/>
 </parts>
 <sheets>
@@
 <instance part="C1" gate="G$1" x="66.04" y="48.26"/>
 <instance part="C2" gate="G$1" x="20.32" y="48.26"/>
-<instance part="L1" gate="G$1" x="58.42" y="53.34"/>
 <instance part="D1" gate="A" x="50.8" y="48.26" rot="R90"/>
 <instance part="SL1" gate="G$1" x="-33.02" y="43.18"/>
@@
 <instance part="D3" gate="1" x="-12.7" y="96.52" rot="R180"/>
 <instance part="C6" gate="G$1" x="2.54" y="81.28"/>
+<instance part="L1" gate="G$1" x="58.42" y="53.34"/>
 </instances>
 <busses>
@@
 <net name="5V" class="0">
 <segment>
-<pinref part="L1" gate="G$1" pin="2"/>
 <wire x1="63.5" y1="53.34" x2="66.04" y2="53.34" width="0.1524" layer="91"/>
 <pinref part="C1" gate="G$1" pin="+"/>
@@
 <wire x1="66.04" y1="53.34" x2="68.58" y2="53.34" width="0.1524" layer="91"/>
 <label x="71.12" y="53.34" size="1.778" layer="95" rot="R90"/>
+<pinref part="L1" gate="G$1" pin="2"/>
 </segment>
 <segment>
@@
 </segment>
 </net>
-<net name="N$2" class="0">
+<net name="LM_OUT" class="0">
 <segment>
-<pinref part="L1" gate="G$1" pin="1"/>
 <pinref part="IC1" gate="G$1" pin="OUT"/>
 <wire x1="53.34" y1="53.34" x2="50.8" y2="53.34" width="0.1524" layer="91"/>
@@
 <wire x1="50.8" y1="53.34" x2="48.26" y2="53.34" width="0.1524" layer="91"/>
 <wire x1="50.8" y1="50.8" x2="50.8" y2="53.34" width="0.1524" layer="91"/>
+<pinref part="L1" gate="G$1" pin="1"/>
 </segment>
 </net>
