File: brick_sorter/Board/psu.brd (EAGLE design)
At the start: 30.1 x 36.8 mm, 14 parts, among them IC1 LM2574N-3.3, IC2-12V 786TV, IC2-6V 786TV

Commit message: Board v2.0
Parts:
- moved L1 51.3 mm to (74.2, 41.7)
- moved C5 15.7 mm to (35.6, 34.8)
- moved C1 15.7 mm to (22.9, 43.7)
- moved D1 15.7 mm to (17.8, 37.3)
- moved D3 15.7 mm to (33.0, 27.2)
- moved C2 15.7 mm to (16.5, 19.6)
- moved C6 15.7 mm to (35.6, 19.6)
- moved D2 15.7 mm to (22.9, 27.2)
- moved IC1 15.7 mm to (16.5, 28.4)
- moved IC2-12V 15.7 mm to (30.5, 27.2)
- moved IC2-6V 15.7 mm to (40.6, 27.2)
- moved C3 15.7 mm to (25.4, 34.8)
- moved C4 15.7 mm to (25.4, 19.6)
- moved SL1 15.7 mm to (25.4, 14.5)
Connections:
- net N$2 renamed LM_OUT
Routing:
- net 5V: track 14.0 -> 59.8 mm, vias 0 -> 1
- net 15V: track 54.0 -> 67.9 mm
- net LM_OUT: track 25.5 -> 24.2 mm, vias 0 -> 1
Other:
- board size 30.1 x 36.8 mm -> 51.5 x 60.4 mm

Commit message: Board v2.1 - now reversed
Routing:
- net N$1: track 0.00 -> 5.90 mm
- net 5V: track 59.8 -> 58.4 mm, vias 1 -> 0
- net 6V: track 19.4 -> 18.6 mm
- net 15V: track 67.9 -> 68.6 mm
- net 12V: track 19.4 -> 18.7 mm
- net LM_OUT: vias 1 -> 0
