File: brick_sorter/Board/led_controller/led.brd (EAGLE design)
At the start: 100 x 80 mm, 17 parts, among them IC1 MAX412CPA, T1 BC547, T2 BC547, T3 BC547

Commit message: Added report and serial console
Parts:
- moved R5 2.84 mm to (50.8, 44.5)
- moved R3 2.54 mm to (45.7, 40.6)
- moved LED3 1.55 mm to (55.6, 50.5), turned to 225 degrees
- moved LED2 0.36 mm to (42.2, 50.5), turned to 225 degrees
Routing:
- net N$5: track 9.94 -> 6.25 mm
- net N$8: track 8.15 -> 4.50 mm
- net 12V: track 90.9 -> 87.6 mm
- net N$10: track 39.5 -> 36.7 mm
- net N$6: track 3.81 -> 5.75 mm
Other:
- board size 100 x 80 mm -> 74.3 x 80.3 mm
- board text added: "B"
- board text added: "G"
- board text added: "R"
