File: brick_sorter/Board/led_controller/led.sch (EAGLE design)
At the start: 17 parts, among them IC1 MAX412CPA, T1 BC547, T2 BC547, T3 BC547

Commit message: Added report and serial console
Changed lines of the file:
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@@
 <pinref part="R2" gate="G$1" pin="1"/>
 <wire x1="20.32" y1="53.34" x2="17.78" y2="53.34" width="0.1524" layer="91"/>
+<label x="10.16" y="53.34" size="1.778" layer="95"/>
 </segment>
 <segment>
@@
 <pinref part="R4" gate="G$1" pin="1"/>
 <wire x1="55.88" y1="53.34" x2="53.34" y2="53.34" width="0.1524" layer="91"/>
+<label x="45.72" y="53.34" size="1.778" layer="95"/>
 </segment>
 <segment>
@@
 <pinref part="R6" gate="G$1" pin="1"/>
 <wire x1="93.98" y1="53.34" x2="91.44" y2="53.34" width="0.1524" layer="91"/>
+<label x="83.82" y="53.34" size="1.778" layer="95"/>
 </segment>
 <segment>
