File: brick_sorter/Board/power_supply/psu.sch (EAGLE design)
At the start: 14 parts, among them IC1 LM2574N-3.3, IC2-12V 786TV, IC2-6V 786TV

Commit message: Updates to report
Parts:
- C1: value (none) -> 330uF
- C2: value (none) -> 22uF
- C3, C4, C5, C6: value (none) -> 330nF
- D1: value BYV10 -> 1N5817
- L1: value (none) -> 330uH
- renumbered IC2-12V to NCP7812TG, IC2-6V to L7806CV
Other:
- moved on the sheet: C1, C2, D1, D2, D3, IC1, L1
